File: MacroPad/Schem and PCB Resources/hackpad.kicad_pcb (KiCad board)
At the start: 2 copper layers, 85.5 x 61 mm, 21 parts, among them J2 Conn_01x04_Pin, SW1 SW_Push_45deg, SW2 SW_Push_45deg, SW3 SW_Push_45deg, SW4 RotaryEncoder_Switch, SW5 SW_Push_45deg, SW6 SW_Push_45deg, SW9 SW_Push_45deg, U1 MOUDLE-SEEEDUINO-XIAO

Commit message: Add files via upload
Finished with the Project! (hope so)
Parts:
- added REF**: MountingHole_2.5mm, MountingHole:MountingHole_2.5mm, F.Cu at (145.7, 62.0)
Changed lines of the file:
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@@
 		(filling no)
 		(pcbplotparams
-			(layerselection 0x00000000_00000000_55555555_5755f5ff)
+			(layerselection 0x00000000_00000000_55557fd5_5fffffff)
 			(plot_on_all_layers_selection 0x00000000_00000000_00000000_00000000)
 			(disableapertmacros no)
@@
 			(outputformat 1)
 			(mirror no)
-			(drillshape 1)
+			(drillshape 0)
 			(scaleselection 1)
-			(outputdirectory "")
+			(outputdirectory "D:/PCB and Models/MacroPad/Production/Gerber FIle/")
 		)
 	)
@@
 		)
 	)
+	(footprint "MountingHole:MountingHole_2.5mm"
+		(layer "F.Cu")
+		(at 145.725 61.975)
+		(descr "Mounting Hole 2.5mm, no annular, generated by kicad-footprint-generator mountinghole.py")
+		(tags "mountinghole")
+		(property "Reference" "REF**"
+			(at 0 -3.45 0)
+			(layer "F.SilkS")
+			(effects
+				(font
+					(size 1 1)
+					(thickness 0.15)
+				)
+			)
+		)
+		(property "Value" "MountingHole_2.5mm"
+			(at 0 3.45 0)
+			(layer "F.Fab")
+			(effects
+				(font
+					(size 1 1)
+					(thickness 0.15)
+				)
+			)
+		)
+		(property "Datasheet" ""
+			(at 0 0 0)
+			(layer "F.Fab")
+			(hide yes)
+			(effects
+				(font
+					(size 1.27 1.27)
+				)
+			)
+		)
+		(property "Description" ""
+			(at 0 0 0)
+			(layer "F.Fab")
+			(hide yes)
+			(effects
+				(font
+					(size 1.27 1.27)
+				)
+			)
+		)
+		(property "KiLib_Generator" "mounting_hardware/mounting_hole"
+			(at 0 0 0)
+			(layer "F.SilkS")
+			(hide yes)
+			(effects
+				(font
+					(size 1 1)
+					(thickness 0.15)
+				)
+			)
+		)
+		(attr exclude_from_pos_files exclude_from_bom)
+		(duplicate_pad_numbers_are_jumpers no)
+		(fp_circle
+			(center 0 0)
+			(end 2.5 0)
+			(stroke
+				(width 0.15)
+				(type solid)
+			)
+			(fill no)
+			(layer "Cmts.User")
+		)
+		(fp_circle
+			(center 0 0)
+			(end 2.75 0)
+			(stroke
+				(width 0.05)
+				(type solid)
+			)
+			(fill no)
+			(layer "F.CrtYd")
+		)
+		(fp_text user "${REFERENCE}"
+			(at 0 0 0)
+			(layer "F.Fab")
+			(effects
+				(font
+					(size 1 1)
+					(thickness 0.15)
+				)
+			)
+		)
+		(pad "" np_thru_hole circle
+			(at 0 0)
+			(size 2.5 2.5)
+			(drill 2.5)
+			(layers "*.Cu" "*.Mask")
+		)
+		(embedded_fonts no)
+	)
 	(footprint "Diode_THT:D_DO-35_SOD27_P7.62mm_Horizontal"

Commit message: Add files via upload
fixed the pcb errors.
Parts:
- D10, D2, D8, D9: footprint LED_SMD:LED_SK6812MINI-E_3.2x2.8mm_P1.5mm_ReverseMount -> LED_SMD:LED_WS2812B_PLCC4_5.0x5.0mm_P3.2mm
- moved D7 65.6 mm to (145.6, 55.5)
- moved D99 20.4 mm to (99.0, 88.7)
- moved D2 7.61 mm to (87.3, 87.6)
- moved D10 4.99 mm to (123.3, 56.7)
- moved D1 3.95 mm to (99.2, 91.7)
- moved D3 3.95 mm to (99.2, 95.2)
- moved D5 3.95 mm to (99.2, 98.8)
- moved D6 3.95 mm to (99.2, 102.3)
- moved REF** 2.79 mm to (102.5, 83.2)
- moved D8 2.67 mm to (87.9, 105.5)
- moved D9 1.63 mm to (163.7, 55.5)
Routing:
- net EC11SWA: track 86.5 -> 14.0 mm
- net Row 1: track 43.9 -> 102.7 mm, vias 1 -> 2
- net Net-(D99-A): track 39.3 -> 13.5 mm, vias 1 -> 0
- net GND: track 178.0 -> 154.6 mm, vias 0 -> 2
- net VCC: track 154.1 -> 133.9 mm
- net Column 3: track 95.8 -> 112.5 mm, vias 1 -> 0
- net Column 2: track 107.0 -> 97.6 mm
- net SDA: track 30.5 -> 22.8 mm
- net Column 1: track 89.0 -> 81.8 mm
- net Row 2: track 47.0 -> 53.9 mm, vias 0 -> 1
- net Net-(D10-DOUT): track 65.6 -> 71.2 mm, vias 2 -> 0
- net Net-(D10-DIN): track 32.0 -> 37.3 mm, vias 2 -> 0
- net EC11SWB: track 66.8 -> 62.0 mm, vias 2 -> 1
- net Net-(D1-A): track 15.0 -> 10.9 mm
- net Net-(D8-DOUT): track 136.8 -> 134.2 mm
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