File: MacroPad/Schem and PCB Resources/hackpad.kicad_sch (KiCad schematic)
At the start: 20 parts, among them J2 Conn_01x04_Pin, SW1 SW_Push_45deg, SW2 SW_Push_45deg, SW3 SW_Push_45deg, SW4 RotaryEncoder_Switch, SW5 SW_Push_45deg, SW6 SW_Push_45deg, SW9 SW_Push_45deg, U1 MOUDLE-SEEEDUINO-XIAO

Commit message: Add files via upload
fixed the pcb errors.
Parts:
- D10, D2, D8, D9: footprint LED_SMD:LED_SK6812MINI-E_3.2x2.8mm_P1.5mm_ReverseMount -> LED_SMD:LED_WS2812B_PLCC4_5.0x5.0mm_P3.2mm
Changed lines of the file:
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@@
 			)
 		)
-		(property "Footprint" "LED_SMD:LED_SK6812MINI-E_3.2x2.8mm_P1.5mm_ReverseMount"
+		(property "Footprint" "LED_SMD:LED_WS2812B_PLCC4_5.0x5.0mm_P3.2mm"
 			(at 62.23 130.81 0)
 			(hide yes)
@@
 			)
 		)
-		(property "Footprint" "LED_SMD:LED_SK6812MINI-E_3.2x2.8mm_P1.5mm_ReverseMount"
+		(property "Footprint" "LED_SMD:LED_WS2812B_PLCC4_5.0x5.0mm_P3.2mm"
 			(at 43.18 130.81 0)
 			(hide yes)
@@
 			)
 		)
-		(property "Footprint" "LED_SMD:LED_SK6812MINI-E_3.2x2.8mm_P1.5mm_ReverseMount"
+		(property "Footprint" "LED_SMD:LED_WS2812B_PLCC4_5.0x5.0mm_P3.2mm"
 			(at 26.67 130.81 0)
 			(hide yes)
@@
 			)
 		)
-		(property "Footprint" "LED_SMD:LED_SK6812MINI-E_3.2x2.8mm_P1.5mm_ReverseMount"
+		(property "Footprint" "LED_SMD:LED_WS2812B_PLCC4_5.0x5.0mm_P3.2mm"
 			(at 76.2 128.27 0)
 			(hide yes)
